File: hardware/main_schematic/sensor-based-mcu.kicad_sch (KiCad schematic)
At the start: 0 parts

Commit message: sensor based mcu
Schematic completed
Parts:
- added IC1: BMP280-module, Sensor:BMP280-module, symbol BMP280-module:2651
- added SENS-1: DHT11, Sensor:SENSOR-DHT11, symbol DHT11:DHT11
- added U1: STM32G071RBIx, Package_BGA:UFBGA-64_5x5mm_Layout8x8_P0.5mm, symbol MCU_ST_STM32G0:STM32G071RBIx
- added U2: Olimex_MOD-WIFI-ESP8266-DEV, Module:Olimex_MOD-WIFI-ESP8266-DEV, symbol MCU_Module:Olimex_MOD-WIFI-ESP8266-DEV
- added U3, U4: ZC362800_, Sensor:BH1750, symbol ZC362800_:ZC362800_
Connections:
- new net: SENS-1.P$2 (DAT), U1.B8 (PA10/PA12)
- new net: IC1.6 (SDI), U1.A3 (PB7)
- new net: IC1.4 (SCK), U1.C8 (PA9/PA11)
- new net: U1.F3 (PA3), U2.19 (GPIO15)
- new net: U1.G3 (PA2), U2.17 (GPIO14)
- new net: IC1.3 (GND), U3.GND, U4.ADDR, U4.GND
- new net: U3.SCL, U4.SCL
- new net: U3.SDA, U4.SDA
- new net 3.3V (from ESP LDO): U2.1 (3.3V)
- new net 3.3V (from Nucleo LDO): IC1.1 (VIN), U1.D1 (VDD), U3.ADDR, U3.VCC, U4.VCC
- new net 5V (from Nucleo): SENS-1.P$1 (VCC)
- new net GND (from ESP LDO): U2.2 (GND)
- new net GND (from Nucleo LDO): SENS-1.P$4 (GND), U1.E1 (VSS)
- no-connect marks 0 -> 23
Other:
- note added: "NUCLEO-G071RB BOARD"
- company: (none) -> Marcel Siwiela

Commit message: info about the project
Parts:
- U3, U4: value ZC362800_ -> BH1750
Changed lines of the file:
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@@
 			)
 		)
-		(property "Value" "ZC362800_"
+		(property "Value" "BH1750"
 			(at 162.56 120.6499 0)
 			(show_name no)
@@
 			)
 		)
-		(property "Value" "ZC362800_"
+		(property "Value" "BH1750"
 			(at 162.56 92.7099 0)
 			(show_name no)
