File: hardware/main_schematic/.history/sensor-based-mcu.kicad_sch (KiCad schematic)
At the start: 6 parts, among them IC1 BMP280-module, U1 STM32G071RBIx, U2 Olimex_MOD-WIFI-ESP8266-DEV, U3 ZC362800_, U4 ZC362800_

Commit message: info about the project
Parts:
- U4: value ZC362800_ -> BH1750
Changed lines of the file:
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@@
 			)
 		)
-		(property "Value" "ZC362800_"
+		(property "Value" "BH1750"
 			(at 162.56 120.6499 0)
 			(show_name no)
